Commit message: gazebo ok

File: air_moveit_config/config/gazebo_air_robot.urdf (robot description, URDF)
Before this commit: robot air_robot, 8 links, 7 joints
Links:
- added link world
Joints:
- added joint world-base_link-fixed: type fixed, parent world, child base_link, origin xyz=0.0 0.0 0.0 rpy=0.0 0.0 0.0

Commit message: gazebo + ROS & ROS + Real HW

File: air_moveit_config/config/gazebo_air_robot.urdf (robot description, URDF)
Before this commit: robot air_robot, 9 links, 8 joints
Joints:
- joint ej: limit lower=-1.4 upper=0.184 effort=0 velocity=0.13 -> lower=-1.4 upper=0.184 effort=2.76 velocity=3.39
- joint pitchj: limit lower=-0.26 upper=0.26 effort=0 velocity=0.09 -> lower=-0.26 upper=0.26 effort=2.76 velocity=3.39
- joint rollj: limit lower=-0.26 upper=0.26 effort=0 velocity=0.09 -> lower=-0.26 upper=0.26 effort=2.76 velocity=3.39
- joint s1j: limit lower=-0.78 upper=0.78 effort=0 velocity=0.35 -> lower=-0.78 upper=0.78 effort=2.76 velocity=3.39
- joint s2j: limit lower=0 upper=1.57 effort=0 velocity=0.35 -> lower=0 upper=1.57 effort=2.76 velocity=3.39
- joint s3j: limit lower=-1.57 upper=1.57 effort=0 velocity=0.35 -> lower=-1.57 upper=1.57 effort=2.76 velocity=3.39
- joint yawj: limit lower=-3.0 upper=3.0 effort=0 velocity=1.75 -> lower=-3.0 upper=3.0 effort=2.76 velocity=3.39
